File: Electrical/MainBoard/MainBoard.kicad_sch (KiCad schematic)
At the start: 0 parts

Commit message: Update KiCAD format
Other:
- company: blame- satomm@stanford.edu -> satomm@stanford.edu

Commit message: Add the majority of the electronics
Parts:
- added C1, C10, C2, C3, C4, C5, C6, C7, C8, C9: 0.1 uF, Capacitor_SMD:C_0805_2012Metric_Pad1.18x1.45mm_HandSolder, symbol Device:C
- added H1, H2, H3, H4: MountingHole, MountingHole:MountingHole_3.2mm_M3, symbol Lab_3:MountingHole
- added J1: SNAP Program, Connector_PinSocket_2.54mm:PinSocket_1x06_P2.54mm_Horizontal, symbol Connector_Generic:Conn_01x06
- added R1: 1k, Resistor_SMD:R_0805_2012Metric_Pad1.20x1.40mm_HandSolder, symbol Device:R_US
- added R2: 10k, Resistor_SMD:R_0805_2012Metric_Pad1.20x1.40mm_HandSolder, symbol Device:R_US
- added SW1: Reset, RobotLibrary:SW_B3F-1000_OMR, symbol RobotLibary:B3F-1020
- added U1: PIC32MZ2048EFH144-I/PL, RobotLibrary:LQFP144_PL_MCH-M, symbol RobotLibary:PIC32MZ2048EFH144-I_PL
Connections:
- new net: J1.2 (Pin_2), U1.35 (PGEC1/AN1/RPB1/RB1)
- new net: J1.3 (Pin_3), U1.36 (PGED1/AN0/RPB0/RB0)
- new net: J1.6 (Pin_6), R1.1, U1.20 (MCLR)
- new net: C10.1, R1.2, R2.1, SW1.4
- new net +3.3V: C1.2, C2.2, C3.2, C4.1, C5.1, C6.1, C7.2, C8.1, C9.1, J1.5 (Pin_5), R2.2, U1.107 (VDD), U1.122 (VDD), U1.137 (VDD), U1.18 (VDD), U1.33 (VDD), U1.41 (AVDD), U1.55 (VDD), U1.64 (VDD), U1.88 (VDD)
- new net Bump1: U1.1 (AN23/RG15)
- new net Bump2: U1.2 (EBIA5/AN34/PMA5/RA5)
- new net Bump3: U1.3 (EBID5/AN17/RPE5/PMD5/RE5)
- new net Bump4: U1.4 (EBID6/AN16/PMD6/RE6)
- new net GND: C1.1, C10.2, C2.1, C3.1, C4.2, C5.2, C6.2, C7.1, C8.2, C9.2, J1.4 (Pin_4), SW1.1, U1.108 (VSS), U1.123 (VSS), U1.136 (VSS), U1.17 (VSS), U1.32 (VSS), U1.42 (AVSS), U1.54 (VSS), U1.63 (VSS), U1.75 (VSS), U1.89 (VSS)
- new net GPS_INT: U1.141 (TRD0/SQID0/RG13)
- new net GPS_Reset: U1.142 (EBID2/PMD2/RE2)
- new net IC1: U1.104 (RPD0/RTCC/INT0/RD0)
- new net IC2: U1.81 (ERXD0/RH8)
- new net IC3: U1.95 (RPA14/SCL1/RA14)
- new net IC4: U1.13 (EBIOE/AN19/RPC4/PMRD/RC4)
- new net IMU_INT1: U1.112 (EBID12/RPD12/PMD12/RD12)
- new net IMU_INT2: U1.113 (EBID13/PMD13/RD13)
- new net LED1: U1.65 (AN40/ERXERR/RH4)
- new net LED2: U1.66 (AN41/ERXD1/RH5)
- new net LED3: U1.67 (AN42/ERXD2/RH6)
- new net LED4: U1.68 (EBIA4/PMA4/RH7)
- new net LED5: U1.71 (OSC1/CLKI/RC12)
- new net LED6: U1.72 (OSC2/CLKO/RC15)
- new net OC1: U1.79 (SDA3/RPF2/RF2)
- new net OC2: U1.119 (SQICS1/RPD5/RD5)
- new net Refl1: U1.5 (EBID7/AN15/PMD7/RE7)
- new net Refl2: U1.6 (EBIA6/AN22/RPC1/PMA6/RC1)
- new net Refl3: U1.7 (AN35/ETXD0/RJ8)
- new net SCK1: U1.109 (RPD1/SCK1/RD1)
- new net SCK2: U1.14 (AN14/C1IND/RPG6/SCK2/RG6)
- new net SCK3: U1.61 (AN9/RPB14/SCK3/RB14)
- new net SCK4: U1.98 (RPD10/SCK4/RD10)
- new net SCK5: U1.57 (TDI/AN30/RPF13/SCK5/RF13)
- new net SCK6: U1.70 (AN33/RPD15/SCK6/RD15)
- new net SDI1: U1.110 (EBID14/RPD2/PMD14/RD2)
- new net SDI2: U1.15 (AN13/C1INC/RPG7/SDA4/RG7)
- new net SDI3: U1.48 (EBIA7/AN49/RPB9/PMA7/RB9)
- new net SDI4: U1.99 (EMDC/RPD11/RD11)
- new net SDI5: U1.127 (EBID9/RPG1/PMD9/RG1)
- new net SDI6: U1.23 (AN25/RPE8/RE8)
- new net SDO1: U1.111 (EBID15/RPD3/PMD15/RD3)
- new net SDO2: U1.16 (AN12/C2IND/RPG8/SCL4/RG8)
- new net SDO3: U1.47 (EBIA10/AN48/RPB8/PMA10/RB8)
- new net SDO4: U1.96 (RPA15/SDA1/RA15)
- new net SDO5: U1.128 (EBID8/RPG0/PMD8/RG0)
- new net SDO6: U1.24 (AN26/RPE9/RE9)
- new net SS1*: U1.118 (SQICS0/RPD4/RD4)
- new net SS2*: U1.21 (EBIA2/AN11/C2INC/RPG9/PMA2/RG9)
- new net SS3*: U1.62 (AN10/RPB15/OCFB/RB15)
- new net SS4*: U1.97 (EBIA15/RPD9/PMCS2/PMA15/RD9)
- new net SS5*: U1.58 (TDO/AN31/RPF12/RF12)
- new net SS6*: U1.69 (AN32/RPD14/RD14)
- new net Status_Green: U1.132 (EBICS1/RJ5)
- new net Status_Yellow: U1.131 (EBICS0/RJ4)
- new net Switch1: U1.82 (ERXD3/RH9)
- new net Switch2: U1.83 (ECOL/RH10)
- new net Switch3: U1.84 (EBIRDY2/RH11)
- new net U1RX: U1.90 (EBIA9/RPF4/SDA5/PMA9/RF4)
- new net U1TX: U1.91 (EBIA8/RPF5/SCL5/PMA8/RF5)
- new net U2RX: U1.143 (EBID3/RPE3/PMD3/RE3)
- new net U2TX: U1.11 (EBIA12/AN21/RPC2/PMA12/RC2)
- new net U3RX: U1.121 (ETXCLK/RPD7/RD7)
- new net U3TX: U1.120 (ETXEN/RPD6/RD6)
- new net U4RX: U1.37 (PGEC2/AN46/RPB6/RB6)
- new net U4TX: U1.38 (PGED2/AN47/RPB7/RB7)
- new net U5RX: U1.25 (AN45/C1INA/RPB5/RB5)
- new net U5TX: U1.31 (AN3/C2INA/RPB3/RB3)
- new net U6RX: U1.34 (AN2/C2INB/RPB2/RB2)
- new net U6TX: U1.12 (EBIWE/AN20/RPC3/PMWR/RC3)
- no-connect marks 0 -> 1
Other:
- added sheet Buttons (Buttons.kicad_sch)
- added sheet GPS (GPS.kicad_sch)
- added sheet IMU (IMU.kicad_sch)
- added sheet LED (LED.kicad_sch)
- added sheet Motor (Motor.kicad_sch)
- added sheet OtherSensors (OtherSensors.kicad_sch)
- added sheet Power (Power.kicad_sch)
- added sheet SPI_UART (SPI_UART.kicad_sch)
- added sheet USB (USB.kicad_sch)
- note added: "Bumper/ Cliff Sensors"
- note added: "Buttons"
- note added: "Figure out antenna"
- note added: "GPS"
- note added: "IMU"
- note added: "LEDs"
- note added: "MCLR"
- note added: "PGEC1"
- note added: "PGED1"
- note added: "Power"
- note added: "SPI/ UART"
- note added: "TODO"
- note added: "USB needs to be taken care of"
- title: Test sheet -> MCU Controller

Commit message: Add more schematics and begin floorplanning
Parts:
- SW1: footprint RobotLibrary:SW_B3F-1000_OMR -> SW_B3F-1000_OMR
Connections:
- net GND: now also U1.74 (VUSB3V3)
- net RH12: now reaches U1.100 (ECRS/RH12)
- net RH13: now reaches U1.101 (ERXDV/ECRSDV/RH13)
- net RH14: now reaches U1.102 (RH14)
- net RH15: now reaches U1.103 (EBIA23/RH15)
- net Dir2: now reaches U1.117 (EBIA22/RJ3)
- net Dir1: now reaches U1.80 (SCL3/RPF8/RF8)
- net SCL2: now reaches U1.85 (SCL2/RA2)
- net SDA2: now reaches U1.86 (EBIRDY1/SDA2/RA3)
- net USB_RST: now reaches U1.92 (EBIA18/RK4)
- net Fault2: now reaches U1.10 (EBIBS1/RJ10)
- net RB4: now reaches U1.26 (AN4/C1INB/RB4)
- net RJ11: now reaches U1.27 (AN37/ERXCLK/EREFCLK/RJ11)
- net RJ13: now reaches U1.28 (EBIA13/PMA13/RJ13)
- net RJ14: now reaches U1.29 (EBIA11/PMA11/RJ14)
- net RJ15: now reaches U1.30 (EBIA0/PMA0/RJ15)
- net RA9: now reaches U1.39 (VREF-/CVREF-/AN27/RA9)
- net RA10: now reaches U1.40 (VREF+/CVREF+/AN28/RA10)
- net RH0: now reaches U1.43 (AN38/ETXD2/RH0)
- net RH1: now reaches U1.44 (AN39/ETXD3/RH1)
- net RH2: now reaches U1.45 (EBIRP/RH2)
- net RH3: now reaches U1.46 (RH3)
- net RB10: now reaches U1.49 (CVREFOUT/AN5/RPB10/RB10)
- net RB11: now reaches U1.50 (AN6/RB11)
- net RK1: now reaches U1.51 (EBIA1/PMA1/RK1)
- net RK2: now reaches U1.52 (EBIA3/PMA3/RK2)
- net RK3: now reaches U1.53 (EBIA17/RK3)
- net MotorCurrent2: now reaches U1.56 (TCK/AN29/RA1)
- net Write Protect*: now reaches U1.59 (AN7/RB12)
- net Hold*: now reaches U1.60 (AN8/RB13)
- net MotorCurrent1: now reaches U1.8 (AN36/ETXD1/RJ9)
- net Fault1: now reaches U1.9 (EBIBS0/RJ12)
- no-connect marks 1 -> 27
Other:
- added sheet GPIO (GPIO.kicad_sch)
- added sheet Memory (Memory.kicad_sch)
- sheet Motor ports: added Dir1, Dir2, Fault1, Fault2, MotorCurrent1, MotorCurrent2; removed none
- sheet SPI_UART ports: added GND, SCK2, SCL2, SDA2, SDI2, SDO2, SS2*; removed SCK5, SCK6, SDI5, SDI6, SDO5, SDO6, SS5*, SS6*, U1RX, U1TX
- sheet USB ports: added 3V3, GND, U1RX, U1TX, USB Reset; removed none
- note added: "GPIO"
- note added: "Memory"
- note added: "Motor Control"
- note added: "SPI/ UART/ I2C"
- note added: "Signal Conditioning?"
- note added: "USB"
- note removed: "SPI/ UART"
- note removed: "TODO"
- note removed: "USB needs to be taken care of"
- moved on the sheet: C2, C3, C8

Commit message: Begin layout of pcb
Parts:
- renumbered C10 to C1, C3 to C10, C8 to C2, C2 to C3, C1 to C4, C9 to C5, C5 to C8, C4 to C9, H3 to H2, H2 to H3, R2 to R1, R1 to R2
Connections:
- net LED1: now also U1.66 (AN41/ERXD1/RH5); no longer U1.65 (AN40/ERXERR/RH4)
- net LED2: now also U1.65 (AN40/ERXERR/RH4); no longer U1.66 (AN41/ERXD1/RH5)
- net LED3: now also U1.68 (EBIA4/PMA4/RH7); no longer U1.67 (AN42/ERXD2/RH6)
- net LED4: now also U1.67 (AN42/ERXD2/RH6); no longer U1.68 (EBIA4/PMA4/RH7)
- net LED5: now also U1.72 (OSC2/CLKO/RC15); no longer U1.71 (OSC1/CLKI/RC12)
- net LED6: now also U1.71 (OSC1/CLKI/RC12); no longer U1.72 (OSC2/CLKO/RC15)
