File: Electrical/MainBoard/MainBoard.kicad_pcb (KiCad board)
At the start: 4 copper layers, 100 x 86.3 mm, 137 parts, among them J1 SNAP Program, J13 Refl_PCB_Connect, J14 Refl_PCB_Connect, J15 Refl_PCB_Connect, J16 Conn_02x03_Odd_Even, J17 MEM2061-01-188-00-A, J18 Conn_02x02_Odd_Even, J19 Conn_02x03_Odd_Even, J2 3.3V Supply, J20 Conn_01x06, J21 Conn_02x03_Odd_Even, J22 Conn_02x02_Odd_Even, J23 Conn_02x03_Odd_Even, J24 Conn_01x04, J25 Conn_02x02_Odd_Even, J26 Conn_02x04_Odd_Even, J3 5V Supply, J4 USB_B_Micro, J5 Battery1, J6 Battery1, J7 GPIO1, J8 Conn_02x04_Odd_Even, J9 USB_B_Micro, SW1 Reset, SW10 SW_SPST, SW2 5V Bypass, SW3 All Power Switch, SW4 User_Button, SW5 User_Button, SW6 User_Button, SW7 SW_SPST, SW8 SW_SPST, SW9 SW_SPST, U1 PIC32MZ2048EFH144-I/PL, U10 DRV8842PWPR, U11 Quad_Encoder_Motor, U12 Quad_Encoder_Motor, U13 DRV8842PWPR, U15 M95M01-DFMN6TP, U2 AP2114HA-3.3TRG1, U3 AP2114HA-3.3TRG1, U5 GSF7002DW, U6 GSF7002DW, U7 GSF7002DW, U8 GSF7002DW, U9 MCP2221A-I_SL

Commit message: Finalize rev 0.2
Routing:
- net +3.3V: track 149.8 -> 148.4 mm
- net GND: track 138.6 -> 137.7 mm
- net /IC4: track 41.1 -> 40.4 mm
Other:
- board text added: "3V3 Int2 Int1 SDO1"
- board text added: "GND SCK1 SS1 SDI1"
- board text added: "IMU"
- board text added: "Matthew Sato, 03/10/2024 Engineering Informatics Group Stanford University Robot Control Board, Rev 0.2"
- board text removed: "Main Power Switch"
- board text removed: "Matthew Sato, 02/02/2024 Engineering Informatics Group Stanford University Robot Control Board, Rev 0.2"
Changed lines of the file:
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@@
   (title_block
     (title "Main Robot Board")
-    (date "2024-02-02")
+    (date "2024-03-10")
     (rev "0.2")
     (company "satomm@stanford.edu")
@@
     (fp_line (start 13.97 2.88) (end 13.97 -2.92)
       (stroke (width 0.1) (type solid)) (layer "F.Fab"))
-    (pad "1" thru_hole roundrect (at 0 0 270) (size 1.74 2.19) (drill 1.19) (layers "*.Cu" "*.Mask") (roundrect_rratio 0.143678)
+    (pad "1" thru_hole roundrect (at 0 0 270) (size 1.74 2.19) (drill 1.19) (layers "*.Cu" "*.Mask") (roundrect_rratio 0.1436781609)
       (net 96 "/IC1") (pinfunction "PhaseA") (pintype "output"))
     (pad "2" thru_hole oval (at 2.54 0 270) (size 1.74 2.19) (drill 1.19) (layers "*.Cu" "*.Mask")
@@
     (fp_line (start 13.97 2.88) (end 13.97 -2.92)
       (stroke (width 0.1) (type solid)) (layer "F.Fab"))
-    (pad "1" thru_hole roundrect (at 0 0 90) (size 1.74 2.19) (drill 1.19) (layers "*.Cu" "*.Mask") (roundrect_rratio 0.143678)
+    (pad "1" thru_hole roundrect (at 0 0 90) (size 1.74 2.19) (drill 1.19) (layers "*.Cu" "*.Mask") (roundrect_rratio 0.1436781609)
       (net 95 "/IC3") (pinfunction "PhaseA") (pintype "output"))
     (pad "2" thru_hole oval (at 2.54 0 90) (size 1.74 2.19) (drill 1.19) (layers "*.Cu" "*.Mask")
@@
     (fp_line (start 13.97 2.88) (end 13.97 -2.92)
       (stroke (width 0.1) (type solid)) (layer "F.Fab"))
-    (pad "1" thru_hole roundrect (at 0 0) (size 1.74 2.19) (drill 1.19) (layers "*.Cu" "*.Mask") (roundrect_rratio 0.143678)
+    (pad "1" thru_hole roundrect (at 0 0) (size 1.74 2.19) (drill 1.19) (layers "*.Cu" "*.Mask") (roundrect_rratio 0.1436781609)
       (net 89 "/SCK2") (pinfunction "Pin_1") (pintype "passive"))
     (pad "2" thru_hole oval (at 2.54 0) (size 1.74 2.19) (drill 1.19) (layers "*.Cu" "*.Mask")
@@
     (descr "Through hole straight pin header, 2x04, 2.54mm pitch, double rows")
     (tags "Through hole pin header THT 2x04 2.54mm double row")
+    (property "Description" "")
+    (property "Mfr" "")
+    (property "Mfr P/N" "")
     (property "Sheetfile" "IMU.kicad_sch")
     (property "Sheetname" "IMU")
+    (property "Supplier 1" "DigiKey")
+    (property "Supplier 1 P/N" "10129381-908001BLF-ND")
+    (property "Supplier 2" "")
+    (property "Supplier 2 P/N" "")
     (property "ki_description" "Generic connector, double row, 02x04, odd/even pin numbering scheme (row 1 odd numbers, row 2 even numbers), script generated (kicad-library-utils/schlib/autogen/connector/)")
     (property "ki_keywords" "connector")
@@
     (property "ki_keywords" "cap capacitor")
     (attr smd)
-    (fp_text reference "C5" (at -0.1 1.45 180) (layer "F.SilkS")
+    (fp_text reference "C5" (at -2 -1.61 180) (layer "F.SilkS")
         (effects (font (size 1 1) (thickness 0.15)))
     )
@@
     (effects (font (size 1 1) (thickness 0.15)) (justify left bottom))
   )
+  (gr_text "3V3\nInt2\nInt1\nSDO1" (at 220.77 114.27) (layer "F.SilkS")
+    (effects (font (size 1 1) (thickness 0.15)) (justify right bottom))
+  )
   (gr_text "5V" (at 202.4 83 -90) (layer "F.SilkS")
     (effects (font (size 1 1) (thickness 0.15)) (justify left bottom))
@@
     (effects (font (size 1 1) (thickness 0.15)) (justify left bottom))
   )
-  (gr_text "Matthew Sato, 02/02/2024\nEngineering Informatics Group\nStanford University\nRobot Control Board, Rev 0.2\n\n" (at 181.975 154.075) (layer "F.SilkS")
+  (gr_text "Matthew Sato, 03/10/2024\nEngineering Informatics Group\nStanford University\nRobot Control Board, Rev 0.2\n\n" (at 181.975 154.075) (layer "F.SilkS")
     (effects (font (size 1 1) (thickness 0.15)) (justify left bottom))
   )
@@
     (effects (font (size 1 1) (thickness 0.15)) (justify left bottom))
   )
-  (gr_text "RH" (at 229.05 115.65) (layer "F.SilkS")
+  (gr_text "RH" (at 239.83 115.61) (layer "F.SilkS")
     (effects (font (size 1 1) (thickness 0.15)) (justify left bottom))
   )
@@
     (effects (font (size 1 1) (thickness 0.15)) (justify left bottom))
   )
+  (gr_text "GND\nSCK1\nSS1\nSDI1" (at 226.45 120.33) (layer "F.SilkS")
+    (effects (font (size 1 1) (thickness 0.15)) (justify left bottom))
+  )
   (gr_text "1" (at 244.6 140.95) (layer "F.SilkS")
     (effects (font (size 1 1) (thickness 0.15)) (justify left bottom))
@@
     (effects (font (size 1 1) (thickness 0.15)) (justify left bottom))
   )
-  (gr_text "Main Power\nSwitch" (at 221.4 108.25) (layer "F.SilkS")
+  (gr_text "IMU" (at 223.675 108.4) (layer "F.SilkS")
     (effects (font (size 1 1) (thickness 0.15)) (justify bottom))
   )
@@
   (segment (start 216.925501 119.6) (end 216.6 119.274499) (width 0.25) (layer "F.Cu") (net 1))
   (segment (start 211.5 118.4375) (end 211.5 119.5) (width 0.25) (layer "F.Cu") (net 1))
-  (segment (start 169.75 128.27) (end 169.25 128.77) (width 0.25) (layer "F.Cu") (net 1))
   (segment (start 249.4 117.6) (end 251.4 115.6) (width 0.25) (layer "F.Cu") (net 1))
   (segment (start 189.575 90.975) (end 189.575 90.55) (width 0.25) (layer "F.Cu") (net 1))
@@
   (segment (start 207.7 146.053888) (end 208.426944 145.326944) (width 0.25) (layer "F.Cu") (net 1))
   (segment (start 263.028401 160.478401) (end 263.05 160.5) (width 0.25) (layer "F.Cu") (net 1))
-  (segment (start 257.2375 123.15) (end 257.05 122.9625) (width 0.25) (layer "F.Cu") (net 1))
   (segment (start 181 134.401654) (end 179.151654 136.25) (width 0.5) (layer "F.Cu") (net 1))
   (segment (start 201.951409 139.85) (end 203.05141 138.749999) (width 0.25) (layer "F.Cu") (net 1))
@@
   (segment (start 217.650001 117.412501) (end 217.650001 121.22405) (width 0.25) (layer "F.Cu") (net 2))
   (segment (start 190 107.55) (end 190.05 107.5) (width 0.25) (layer "F.Cu") (net 2))
-  (segment (start 261.385 120.975) (end 261.75 120.61) (width 0.25) (layer "F.Cu") (net 2))
   (segment (start 233.3 132.25) (end 232.0875 132.25) (width 0.25) (layer "F.Cu") (net 2))
   (segment (start 261.050354 110.650353) (end 261.050354 109.487146) (width 0.25) (layer "F.Cu") (net 2))
   (segment (start 247.249998 135.425) (end 245.625 135.425) (width 0.25) (layer "F.Cu") (net 2))
-  (segment (start 257.05 120.8875) (end 257.1375 120.975) (width 0.25) (layer "F.Cu") (net 2))
   (segment (start 208.5 144.3) (end 208.55 144.3) (width 0.25) (layer "F.Cu") (net 2))
   (segment (start 188.85 111.55) (end 190.1 111.55) (width 0.25) (layer "F.Cu") (net 2))
@@
   (segment (start 215.65 143.929057) (end 216.450001 144.729058) (width 0.25) (layer "F.Cu") (net 2))
   (segment (start 206.0242 100.3) (end 203.7375 100.3) (width 0.5) (layer "F.Cu") (net 2))
-  (segment (start 169.8525 130.7075) (end 169.25 131.31) (width 0.25) (layer "F.Cu") (net 2))
   (segment (start 203.6 101.6) (end 203.6 101.8) (width 0.5) (layer "F.Cu") (net 2))
   (segment (start 202.85 132.7) (end 200.1125 132.7) (width 0.25) (layer "F.Cu") (net 2))
@@
   (segment (start 186.644776 137.8) (end 174.3 137.8) (width 0.25) (layer "F.Cu") (net 88))
   (segment (start 199.241962 129.0005) (end 197.167462 131.075) (width 0.25) (layer "F.Cu") (net 88))
-  (segment (start 169.85 133.35) (end 169.1 133.35) (width 0.25) (layer "F.Cu") (net 88))
   (segment (start 200.929095 129.25) (end 200.679595 129.0005) (width 0.25) (layer "F.Cu") (net 88))
   (segment (start 172.055 142.789314) (end 172.055 141.32) (width 0.25) (layer "F.Cu") (net 89))
@@
   (via (at 233.85 136.9255) (size 0.8) (drill 0.4) (layers "F.Cu" "B.Cu") (net 94))
   (segment (start 234.3755 136.4) (end 243.42 136.4) (width 0.25) (layer "B.Cu") (net 94))
-  (segment (start 261.71 118.11) (end 261.925 118.11) (width 0.25) (layer "B.Cu") (net 94))
   (segment (start 233.85 136.9255) (end 234.3755 136.4) (width 0.25) (layer "B.Cu") (net 94))
   (segment (start 243.42 136.4) (end 261.71 118.11) (width 0.25) (layer "B.Cu") (net 94))
@@
   (segment (start 230.299527 125.0755) (end 230.125026 125.250001) (width 0.25) (layer "F.Cu") (net 96))
   (via (at 230.299527 125.0755) (size 0.8) (drill 0.4) (layers "F.Cu" "B.Cu") (net 96))
-  (segment (start 261.75 115.745) (end 261.75 115.53) (width 0.25) (layer "B.Cu") (net 96))
   (segment (start 230.299527 125.0755) (end 231.125027 124.25) (width 0.25) (layer "B.Cu") (net 96))
   (segment (start 231.125027 124.25) (end 253.245 124.25) (width 0.25) (layer "B.Cu") (net 96))
@@
   (segment (start 169.175 114.75) (end 169.175 123.115) (width 0.5) (layer "F.Cu") (net 133))
   (segment (start 177.650001 112.9) (end 171.025 112.9) (width 0.5) (layer "F.Cu") (net 133))
-  (segment (start 169.175 123.115) (end 169.1 123.19) (width 0.5) (layer "F.Cu") (net 133))
   (segment (start 177.650001 112.9) (end 177.650001 113.225) (width 0.5) (layer "F.Cu") (net 133))
   (segment (start 171.025 112.9) (end 169.175 114.75) (width 0.5) (layer "F.Cu") (net 133))
@@
   (segment (start 258.45 133.85) (end 258.45 129.205) (width 0.5) (layer "F.Cu") (net 134))
   (segment (start 253.349999 139.325) (end 253.349999 138.674998) (width 0.5) (layer "F.Cu") (net 135))
-  (segment (start 261.85 128.345) (end 261.925 128.27) (width 0.5) (layer "F.Cu") (net 135))
   (segment (start 255.5 139) (end 259.098439 139) (width 0.5) (layer "F.Cu") (net 135))
   (segment (start 253.349999 139.325) (end 253.6495 139.025499) (width 0.5) (layer "F.Cu") (net 135))
