File: Electrical/MainBoard/Motor.kicad_sch (KiCad schematic)
At the start: 44 parts, among them J27 Conn_01x06_Socket, U1 DRV8842PWPR, U11 Quad_Encoder_Motor, U12 Quad_Encoder_Motor

Commit message: Fix SPI3 and make visual improvements
Parts:
- renumbered C6 to C20, C1 to C21, C4 to C22, C4 to C23, C4 to C24, C3 to C25, C6 to C26, C5 to C27, C5 to C28, C1 to C29, C4 to C30, C4 to C31, C4 to C32, C3 to C33, J27 to J28, J27 to J29, R8 to R17, R9 to R18, R10 to R19, R3 to R20, R3 to R21, R3 to R22, R3 to R23, R3 to R24, R2 to R25, R1 to R26, R8 to R27, R9 to R28, R10 to R29, R3 to R30, R3 to R31, R3 to R32, R3 to R33, R3 to R34, R2 to R35, R1 to R36, R1 to R47, R1 to R48, R1 to R49, R1 to R50, U1 to U10, U1 to U13
Other:
- note added: "Corresponding Molex for Motor Connector: Corresponding Female: DigiKey PN WM2002-ND Corresponding Crimp : DigiKey PN WM2756CT-ND"
- note added: "Left Motor Driver"
- note added: "Motor Connector"
- note added: "Motor Driver"
- note added: "Right Motor Driver"
- note removed: "Corresponding Female: DigiKey PN WM2002-ND Corresponding Crimp : DigiKey PN WM2756CT-ND"
- moved on the sheet: C20, C21, C22, C23, C24, C25, C26, C27, C28, C29, C30, C31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

Commit message: Add updated gerbers
Other:
- moved on the sheet: C22, C23, R17, R18, R19, R20, R21, R22, R23, R24

Commit message: Update some parts
Parts:
- C21, C29: Mfr Samsung Electro-Mechanics -> KEMET; Mfr P/N CL21B103KBANNNC -> C0805C103K5RACTU; Supplier 1 P/N 1276-1015-1-ND -> 399-C0805C103K5RACTUCT-ND
Changed lines of the file:
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@@
 			)
 		)
-		(property "Datasheet" "https://www.samsungsem.com/kr/support/product-search/mlcc/CL21B103KBANNNC.jsp"
+		(property "Datasheet" "https://search.kemet.com/download/datasheet/C0805C103K5RAC7800"
 			(at 314.96 93.98 0)
 			(effects
@@
 			)
 		)
-		(property "Mfr" "Samsung Electro-Mechanics"
+		(property "Mfr" "KEMET"
 			(at 314.96 93.98 0)
 			(effects
@@
 			)
 		)
-		(property "Mfr P/N" "CL21B103KBANNNC"
+		(property "Mfr P/N" "C0805C103K5RACTU"
 			(at 314.96 93.98 0)
 			(effects
@@
 			)
 		)
-		(property "Supplier 1 P/N" "1276-1015-1-ND"
+		(property "Supplier 1 P/N" "399-C0805C103K5RACTUCT-ND"
 			(at 314.96 93.98 0)
 			(effects
@@
 			)
 		)
-		(property "Datasheet" "https://www.samsungsem.com/kr/support/product-search/mlcc/CL21B103KBANNNC.jsp"
+		(property "Datasheet" "https://search.kemet.com/download/datasheet/C0805C103K5RAC7800"
 			(at 113.03 95.25 0)
 			(effects
@@
 			)
 		)
-		(property "Mfr" "Samsung Electro-Mechanics"
+		(property "Mfr" "KEMET"
 			(at 113.03 95.25 0)
 			(effects
@@
 			)
 		)
-		(property "Mfr P/N" "CL21B103KBANNNC"
+		(property "Mfr P/N" "C0805C103K5RACTU"
 			(at 113.03 95.25 0)
 			(effects
@@
 			)
 		)
-		(property "Supplier 1 P/N" "1276-1015-1-ND"
+		(property "Supplier 1 P/N" "399-C0805C103K5RACTUCT-ND"
 			(at 113.03 95.25 0)
 			(effects
