File: Electrical/MainBoard/USB.kicad_sch (KiCad schematic)
At the start: 7 parts, among them J9 USB_B_Micro, U9 MCP2221A-I_SL

Commit message: Update some parts
Parts:
- D10, D9: Mfr Würth Elektronik -> Harvatek Corporation; Mfr P/N 150080RS75000 -> B1701URO-20D000114U1930; Supplier 1 P/N 732-4984-1-ND -> 3147-B1701URO-20D000114U1930CT-ND
Changed lines of the file:
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@@
 			)
 		)
-		(property "Datasheet" "https://www.we-online.com/katalog/datasheet/150080RS75000.pdf"
+		(property "Datasheet" "https://mm.digikey.com/Volume0/opasdata/d220001/medias/docus/3739/B1701URO-20D000114U1930.pdf"
 			(at 258.445 120.015 0)
 			(effects
@@
 			)
 		)
-		(property "Description" "LED RED CLEAR 0805 SMD"
+		(property "Description" "LED RED DIFFUSED 0805 SMD"
 			(at 258.445 120.015 0)
 			(effects
@@
 			)
 		)
-		(property "Mfr" "Würth Elektronik"
+		(property "Mfr" "Harvatek Corporation"
 			(at 258.445 120.015 0)
 			(effects
@@
 			)
 		)
-		(property "Mfr P/N" "150080RS75000"
+		(property "Mfr P/N" "B1701URO-20D000114U1930"
 			(at 258.445 120.015 0)
 			(effects
@@
 			)
 		)
-		(property "Supplier 1 P/N" "732-4984-1-ND"
+		(property "Supplier 1 P/N" "3147-B1701URO-20D000114U1930CT-ND"
 			(at 258.445 120.015 0)
 			(effects
@@
 			)
 		)
-		(property "Datasheet" "https://www.we-online.com/katalog/datasheet/150080RS75000.pdf"
+		(property "Datasheet" "https://mm.digikey.com/Volume0/opasdata/d220001/medias/docus/3739/B1701URO-20D000114U1930.pdf"
 			(at 257.81 123.825 0)
 			(effects
@@
 			)
 		)
-		(property "Description" "LED RED CLEAR 0805 SMD"
+		(property "Description" "LED RED DIFFUSED 0805 SMD"
 			(at 257.81 123.825 0)
 			(effects
@@
 			)
 		)
-		(property "Mfr" "Würth Elektronik"
+		(property "Mfr" "Harvatek Corporation"
 			(at 257.81 123.825 0)
 			(effects
@@
 			)
 		)
-		(property "Mfr P/N" "150080RS75000"
+		(property "Mfr P/N" "B1701URO-20D000114U1930"
 			(at 257.81 123.825 0)
 			(effects
@@
 			)
 		)
-		(property "Supplier 1 P/N" "732-4984-1-ND"
+		(property "Supplier 1 P/N" "3147-B1701URO-20D000114U1930CT-ND"
 			(at 257.81 123.825 0)
 			(effects
