File: Electrical/Archives/V0.3/GPS.kicad_sch (KiCad schematic)
At the start: 4 parts, among them J24 Conn_01x04, U14 MAX-M8C-0

Commit message: Finalize the PCBs
Parts:
- J24: now left out of the parts list
Changed lines of the file:
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@@
 		(unit 1)
 		(exclude_from_sim no)
-		(in_bom yes)
+		(in_bom no)
 		(on_board yes)
 		(dnp no)
