File: Electrical/Archives/V0.3/LED.kicad_sch (KiCad schematic)
At the start: 19 parts, among them U5 GSF7002DW, U6 GSF7002DW, U7 GSF7002DW, U8 GSF7002DW

Commit message: Finalize the PCBs
Parts:
- removed D8: Status_LED, RobotLibrary:CONN3_22232031_MOL, symbol Device:LED_Dual_AKA
- added D11: Status_LED, RobotLibrary:CONN3_22232031_MOL, symbol Device:LED_Dual_KAK
Connections:
- net +3.3V: now also D11.2 (A); no longer U8.3 (D2), U8.6 (D1)
- net GND: now also U8.1 (S1), U8.4 (S2)
- net at R10.1: now also U8.6 (D1)
- net at R10.2: now also D11.3 (K2); no longer U8.1 (S1)
- net at R11.2: now also D11.1 (K1); no longer U8.4 (S2)
- net at R11.1: now also U8.3 (D2)
Other:
- note added: "Corresponding Male : DigiKey PN WM4201-ND Corresponding Female: DigiKey PN 900-0022013037-ND Corresponding Crimp : DigiKey PN WM2756CT-ND"
- note added: "Green"
- note added: "Red"
- note removed: "Corresponding Female: DigiKey PN 900-0022013037-ND Corresponding Crimp : DigiKey PN WM2756CT-ND"
- moved on the sheet: R10, R11, U8
