File: Electrical/Archives/V0.3/MainBoard.kicad_pcb (KiCad board)
At the start: 4 copper layers, 100 x 86.3 mm, 137 parts, among them J1 SNAP Program, J13 Refl_PCB_Connect, J14 Refl_PCB_Connect, J15 Refl_PCB_Connect, J16 Conn_02x03_Odd_Even, J17 MEM2061-01-188-00-A, J18 Conn_02x02_Odd_Even, J19 Conn_02x03_Odd_Even, J2 3.3V Supply, J20 Conn_01x06, J21 Conn_02x03_Odd_Even, J22 Conn_02x02_Odd_Even, J23 Conn_02x03_Odd_Even, J24 Conn_01x04, J25 Conn_02x02_Odd_Even, J26 Conn_02x04_Odd_Even, J3 5V Supply, J4 USB_B_Micro, J5 Battery1, J6 Battery1, J7 GPIO1, J8 Conn_02x04_Odd_Even, J9 USB_B_Micro, SW1 Reset, SW10 SW_SPST, SW2 5V Bypass, SW3 All Power Switch, SW4 User_Button, SW5 User_Button, SW6 User_Button, SW7 SW_SPST, SW8 SW_SPST, SW9 SW_SPST, U1 PIC32MZ2048EFH144-I/PL, U10 DRV8842PWPR, U11 Quad_Encoder_Motor, U12 Quad_Encoder_Motor, U13 DRV8842PWPR, U15 M95M01-DFMN6TP, U2 AP2114HA-3.3TRG1, U3 AP2114HA-3.3TRG1, U5 GSF7002DW, U6 GSF7002DW, U7 GSF7002DW, U8 GSF7002DW, U9 MCP2221A-I_SL

Commit message: Finalize the PCBs
Parts:
- removed D8: Status_LED, RobotLibrary:CONN3_22232031_MOL
- added D11: Status_LED, RobotLibrary:CONN3_22232031_MOL, F.Cu at (206.7, 106.2)
- R10, R11, R15, R16, U8: moved to B.Cu
- moved R16 23.3 mm to (258.5, 116.7)
- moved R15 15.2 mm to (260.6, 106.0)
- moved C28 6.23 mm to (256.9, 128.2)
- moved U11 6.23 mm to (261.8, 121.8)
- moved U9 5.60 mm to (258.2, 109.3)
- moved C19 5.60 mm to (260.1, 115.0)
- moved D10 5.60 mm to (264.4, 114.1)
- moved D9 5.60 mm to (264.4, 107.6)
- moved J9 5.60 mm to (263.9, 100.0)
- moved R10 5.02 mm to (214.4, 107.0), turned to 90 degrees
- moved U8 2.91 mm to (213.5, 110.5)
- moved R11 2.38 mm to (207.5, 108.5), turned to 180 degrees
- moved C24 1.10 mm to (186.9, 122.8)
- moved C1 0.65 mm to (196.1, 128.2)
- moved J5 0.11 mm to (250.0, 101.0)
Connections:
- R10 pad 1: Net-(D8-A1) -> Net-(U8-D1)
- R10 pad 2: Net-(U8-S1) -> Net-(D11-K2)
- R11 pad 1: Net-(D8-A2) -> Net-(U8-D2)
- R11 pad 2: Net-(U8-S2) -> Net-(D11-K1)
- U8 pad 1: Net-(U8-S1) -> GND
- U8 pad 3: +3.3V -> Net-(U8-D2)
- U8 pad 4: Net-(U8-S2) -> GND
- U8 pad 6: +3.3V -> Net-(U8-D1)
Routing:
- net Net-(U8-S2): track 17.0 -> 0.00 mm
- net Net-(D10-A): track 22.5 -> 6.08 mm, vias 2 -> 1
- net Net-(D9-A): track 13.5 -> 3.12 mm, vias 2 -> 1
- net Vdrive: track 208.4 -> 198.5 mm
- net Net-(U8-S1): track 9.83 -> 0.00 mm
- net /USB_RST: track 53.7 -> 45.0 mm, vias 0 -> 2
- net Net-(U11-M-): track 18.3 -> 12.2 mm
- net Net-(U11-M+): track 21.5 -> 16.1 mm
- net Net-(D8-A2): track 4.71 -> 0.00 mm
- net Net-(U8-D2): track 0.00 -> 4.61 mm
- net Net-(D8-A1): track 4.28 -> 0.00 mm
- net Net-(U8-D1): track 0.00 -> 4.04 mm
- net Net-(D11-K2): track 0.00 -> 3.65 mm
- net Net-(D11-K1): track 0.00 -> 2.83 mm
- net /IC2: track 43.6 -> 41.1 mm
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Other:
- board text added: "Matthew Sato, 06/11/2025 Engineering Informatics Group Stanford University Robot Control Board, Rev 0.3 Schematic Details: https://github.com/satomm1/Robot"
- board text added: "NiMH Batt."
- board text added: "R|3V3|G"
- board text removed: "Matthew Sato, 05/18/2025 Engineering Informatics Group Stanford University Robot Control Board, Rev 0.3 Schematic Details: https://github.com/satomm1/Robot"
- board text removed: "Y|GND|G"
