File: Electrical/Archives/V0.3/Memory.kicad_sch (KiCad schematic)
At the start: 4 parts, among them J17 MEM2061-01-188-00-A, U15 M95M01-DFMN6TP

Commit message: Finalize the PCBs
Parts:
- C35, J17: now in the parts list
Changed lines of the file:
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@@
 		(unit 1)
 		(exclude_from_sim no)
-		(in_bom no)
+		(in_bom yes)
 		(on_board yes)
 		(dnp no)
@@
 		(unit 1)
 		(exclude_from_sim no)
-		(in_bom no)
-		(on_board yes)
-		(dnp no)
+		(in_bom yes)
+		(on_board yes)
+		(dnp no)
