File: Electrical/Archives/V0.3/Motor.kicad_sch (KiCad schematic)
At the start: 44 parts, among them J28 Conn_01x06_Socket, J29 Conn_01x06_Socket, U10 DRV8842PWPR, U11 Quad_Encoder_Motor, U12 Quad_Encoder_Motor, U13 DRV8842PWPR

Commit message: Finalize the PCBs
Parts:
- U11, U12: Mfr P/N 0022272061 -> 0022232061; Supplier 1 P/N WM4115-ND -> WM4204-ND
Changed lines of the file:
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@@
 			)
 		)
-		(property "Mfr P/N" "0022272061"
+		(property "Mfr P/N" "0022232061"
 			(at 189.23 62.865 0)
 			(effects
@@
 			)
 		)
-		(property "Supplier 1 P/N" "WM4115-ND"
+		(property "Supplier 1 P/N" "WM4204-ND"
 			(at 189.23 62.865 0)
 			(effects
@@
 			)
 		)
-		(property "Mfr P/N" "0022272061"
+		(property "Mfr P/N" "0022232061"
 			(at 380.365 60.96 0)
 			(effects
@@
 			)
 		)
-		(property "Supplier 1 P/N" "WM4115-ND"
+		(property "Supplier 1 P/N" "WM4204-ND"
 			(at 380.365 60.96 0)
 			(effects
