File: Electrical/Archives/V0.3/Power.kicad_sch (KiCad schematic)
At the start: 17 parts, among them J2 3.3V Supply, J3 5V Supply, J4 USB_B_Micro, J5 Battery1, J6 Battery1, SW2 5V Bypass, SW3 All Power Switch, U2 AP2114HA-3.3TRG1, U3 AP2114HA-3.3TRG1

Commit message: Finalize the PCBs
Other:
- note added: "Molex + Switch Male, DigiKey P/N: WM4622-ND Female, DigiKey P/N: WM2124-ND Crimp, DigiKey P/N: WM20948CT-ND 5A Fuse, DigiKey P/N: F1725-ND"
- note removed: "Molex + Switch Female, DigiKey P/N: WM2124-ND Crimp, DigiKey P/N: WM20948CT-ND"
Changed lines of the file:
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@@
 		)
 	)
-	(text "Molex + Switch\n\nFemale, DigiKey P/N: WM2124-ND\nCrimp,  DigiKey P/N: WM20948CT-ND"
+	(text "Molex + Switch\n\nMale, DigiKey P/N: WM4622-ND\nFemale, DigiKey P/N: WM2124-ND\nCrimp,  DigiKey P/N: WM20948CT-ND\n\n5A Fuse, DigiKey P/N: F1725-ND"
 		(exclude_from_sim no)
-		(at 289.56 173.355 0)
+		(at 288.29 178.435 0)
 		(effects
 			(font
