File: Electrical/Archives/V0.3/SPI_UART.kicad_sch (KiCad schematic)
At the start: 7 parts, among them J18 Conn_02x02_Odd_Even, J19 Conn_02x03_Odd_Even, J20 Conn_01x06, J22 Conn_02x02_Odd_Even, J23 Conn_02x03_Odd_Even, J27 Conn_01x06_Socket, J8 Conn_02x04_Odd_Even

Commit message: Finalize the PCBs
Parts:
- J20: Mfr P/N 0022272061 -> 0022232061; Supplier 1 P/N WM4115-ND -> WM4204-ND
Changed lines of the file:
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@@
 			)
 		)
-		(property "Mfr P/N" "0022272061"
+		(property "Mfr P/N" "0022232061"
 			(at 163.576 124.206 0)
 			(effects
@@
 			)
 		)
-		(property "Supplier 1 P/N" "WM4115-ND"
+		(property "Supplier 1 P/N" "WM4204-ND"
 			(at 163.576 124.206 0)
 			(effects
